File: Proyecto Final/NIVARA/DRIVER-RS485.kicad_sch (KiCad schematic)
At the start: 1 part, among them U3 MAX3485

Commit message: Actualización.
Parts:
- removed U3: MAX3485, Package_SO:SOIC-8_3.9x4.9mm_P1.27mm, symbol Interface_UART:MAX3485
- added C7: C_1206, PCM_Capacitor_SMD_AKL:C_1206_3216Metric, symbol PCM_Capacitor_AKL:C_1206
- added D1: SM712, PCM_Package_TO_SOT_SMD_AKL:SOT-23, symbol PCM_Diode_TVS_AKL:SM712
- added U4: ~, Package_DIP:C2992406, symbol Interface_UART:C2992406
Connections:
- net +3.3V: now also C7.1, U4.1 (VCC)
- net GND: now also C7.2, U4.2 (GND)
- net GPIO Control: now also U4.5 (CON)
- net RS485-A: now also U4.9 (A)
- net RS485-B: now also U4.8 (B)
- net UART_IN: now also U4.3 (TXD)
- net UART_OUT: now also U4.4 (RXD)
Other:
- note removed: "OPTOCOPLAR"

Commit message: Actualización
Connections:
- net +3.3V: now also D1.2 (A2)
- net GND: now also D1.1 (A1), D1.3 (Com)
Other:
- moved on the sheet: D1
Changed lines of the file:
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@@
 	(paper "USLedger")
+	(junction
+		(at 55.88 44.45)
+		(diameter 0)
+		(color 0 0 0 0)
+	)
+	(junction
+		(at 55.88 34.29)
+		(diameter 0)
+		(color 0 0 0 0)
+	)
 	(junction
 		(at 62.23 44.45)
@@
 	(wire
 		(pts
-			(xy 68.58 50.8) (xy 73.66 50.8)
+			(xy 30.48 40.64) (xy 30.48 39.37)
 		)
 		(stroke
@@
 	(wire
 		(pts
-			(xy 72.39 39.37) (xy 73.66 39.37)
+			(xy 55.88 44.45) (xy 62.23 44.45)
 		)
 		(stroke
@@
 	(wire
 		(pts
-			(xy 72.39 34.29) (xy 72.39 39.37)
+			(xy 55.88 34.29) (xy 62.23 34.29)
 		)
 		(stroke
@@
 	(wire
 		(pts
-			(xy 62.23 34.29) (xy 72.39 34.29)
+			(xy 68.58 50.8) (xy 73.66 50.8)
 		)
 		(stroke
@@
 	(wire
 		(pts
-			(xy 52.07 34.29) (xy 52.07 33.02)
+			(xy 55.88 36.83) (xy 55.88 34.29)
 		)
 		(stroke
@@
 	(wire
 		(pts
-			(xy 52.07 44.45) (xy 62.23 44.45)
+			(xy 72.39 39.37) (xy 73.66 39.37)
 		)
 		(stroke
@@
 	(wire
 		(pts
-			(xy 68.58 46.99) (xy 73.66 46.99)
+			(xy 72.39 34.29) (xy 72.39 39.37)
 		)
 		(stroke
@@
 	(wire
 		(pts
-			(xy 72.39 44.45) (xy 72.39 43.18)
+			(xy 62.23 34.29) (xy 72.39 34.29)
 		)
 		(stroke
@@
 	(wire
 		(pts
-			(xy 62.23 34.29) (xy 62.23 35.56)
+			(xy 49.53 41.91) (xy 55.88 41.91)
 		)
 		(stroke
@@
 	(wire
 		(pts
-			(xy 95.25 50.8) (xy 99.06 50.8)
+			(xy 55.88 41.91) (xy 55.88 44.45)
 		)
 		(stroke
@@
 	(wire
 		(pts
-			(xy 95.25 43.18) (xy 99.06 43.18)
+			(xy 52.07 34.29) (xy 52.07 33.02)
 		)
 		(stroke
@@
 	(wire
 		(pts
-			(xy 52.07 34.29) (xy 62.23 34.29)
+			(xy 52.07 44.45) (xy 55.88 44.45)
+		)
+		(stroke
+			(width 0)
+			(type default)
+		)
+	)
+	(wire
+		(pts
+			(xy 68.58 46.99) (xy 73.66 46.99)
+		)
+		(stroke
+			(width 0)
+			(type default)
+		)
+	)
+	(wire
+		(pts
+			(xy 72.39 44.45) (xy 72.39 43.18)
+		)
+		(stroke
+			(width 0)
+			(type default)
+		)
+	)
+	(wire
+		(pts
+			(xy 62.23 34.29) (xy 62.23 35.56)
+		)
+		(stroke
+			(width 0)
+			(type default)
+		)
+	)
+	(wire
+		(pts
+			(xy 30.48 39.37) (xy 34.29 39.37)
+		)
+		(stroke
+			(width 0)
+			(type default)
+		)
+	)
+	(wire
+		(pts
+			(xy 95.25 50.8) (xy 99.06 50.8)
+		)
+		(stroke
+			(width 0)
+			(type default)
+		)
+	)
+	(wire
+		(pts
+			(xy 95.25 43.18) (xy 99.06 43.18)
+		)
+		(stroke
+			(width 0)
+			(type default)
+		)
+	)
+	(wire
+		(pts
+			(xy 52.07 34.29) (xy 55.88 34.29)
+		)
+		(stroke
+			(width 0)
+			(type default)
+		)
+	)
+	(wire
+		(pts
+			(xy 49.53 36.83) (xy 55.88 36.83)
 		)
 		(stroke
@@
 	(symbol
 		(lib_id "PCM_Diode_TVS_AKL:SM712")
-		(at 39.37 39.37 0)
+		(at 41.91 39.37 0)
 		(unit 1)
 		(exclude_from_sim no)
@@
 		(fields_autoplaced yes)
 		(property "Reference" "D1"
-			(at 38.7985 29.21 0)
+			(at 41.3385 29.21 0)
 			(effects
 				(font
@@
 		)
 		(property "Value" "SM712"
-			(at 38.7985 31.75 0)
+			(at 41.3385 31.75 0)
 			(effects
 				(font
@@
 		)
 		(property "Footprint" "PCM_Package_TO_SOT_SMD_AKL:SOT-23"
-			(at 39.37 30.48 0)
+			(at 41.91 30.48 0)
 			(effects
 				(font
@@
 		)
 		(property "Datasheet" "https://www.tme.eu/Document/75933fc1842e5f5f3391c0542bf992c7/SM712.pdf"
-			(at 39.37 30.48 0)
+			(at 41.91 30.48 0)
 			(effects
 				(font
@@
 		)
 		(property "Description" "SOT-23 Dual bidirectional TVS diode, 12V/7V, 600W, Alternate KiCAD Library"
-			(at 39.37 39.37 0)
+			(at 41.91 39.37 0)
 			(effects
 				(font
@@
 					(unit 1)
 				)
+			)
+		)
+	)
+	(symbol
+		(lib_id "power:GND")
+		(at 30.48 40.64 0)
+		(unit 1)
+		(exclude_from_sim no)
+		(in_bom yes)
+		(on_board yes)
+		(dnp no)
+		(fields_autoplaced yes)
+		(property "Reference" "#PWR023"
+			(at 30.48 46.99 0)
+			(effects
+				(font
+					(size 1.27 1.27)
+				)
+				(hide yes)
+			)
+		)
+		(property "Value" "GND"
+			(at 30.48 45.72 0)
+			(effects
+				(font
+					(size 1.27 1.27)
+				)
+			)
+		)
+		(property "Footprint" ""
+			(at 30.48 40.64 0)
+			(effects
+				(font
+					(size 1.27 1.27)
+				)
+				(hide yes)
+			)
+		)
+		(property "Datasheet" ""
+			(at 30.48 40.64 0)
+			(effects
+				(font
+					(size 1.27 1.27)
+				)
+				(hide yes)
+			)
+		)
+		(property "Description" "Power symbol creates a global label with name \"GND\" , ground"
+			(at 30.48 40.64 0)
+			(effects
+				(font
+					(size 1.27 1.27)
+				)
+				(hide yes)
+			)
+		)
+		(pin "1"
+		)
+		(instances
+			(project "PLC"
+				(path "/a1baea3f-df2c-4fcc-baf4-2ec71e099e23/26c5c8f2-e377-4319-a69c-d69661c7cccb/99c91700-32e4-4af2-92bb-dfc39d4a19be"
+					(reference "#PWR023")
+					(unit 1)
+				)
