File: Proyecto Final/NIVARA/Imput_NPN.kicad_sch (KiCad schematic)
At the start: 0 parts

Commit message: Actualización
Parts:
- added D3: DL4007, PCM_Diode_SMD_AKL:D_MELF, symbol PCM_Diode_AKL:DL4007
- added OC1: LTV-357T-B, PCM_Package_SO_AKL:SO-4_4.4x3.9mm_P2.54mm, symbol PCM_Optocoupler_AKL:LTV-357T-B
- added R3, R5: R_0603, PCM_Resistor_SMD_AKL:R_0603_1608Metric, symbol PCM_Resistor_US_AKL:R_0603
Connections:
- new net: D3.1 (K), OC1.1, R3.2
- new net + NPN_IN +: R3.1
- new net +3.3V: R5.2
- new net - NPN_IN -: D3.2 (A), OC1.2
- new net GND: OC1.3
- new net NPN-DInput: OC1.4, R5.1

Commit message: Actualización
Parts:
- added D9: DL4007, PCM_Diode_SMD_AKL:D_MELF, symbol PCM_Diode_AKL:DL4007
- added OC5: LTV-357T-B, PCM_Package_SO_AKL:SO-4_4.4x3.9mm_P2.54mm, symbol PCM_Optocoupler_AKL:LTV-357T-B
- added R18, R19: R_0603, PCM_Resistor_SMD_AKL:R_0603_1608Metric, symbol PCM_Resistor_US_AKL:R_0603
Connections:
- net - NPN_IN - is gone; now on net GND: D3.2 (A), OC1.2
- net +3.3V: now also R19.2
- net GND: now also D9.2 (A), OC5.2, OC5.3
- net + NPN_IN + renamed NPN_IN-1
- net NPN-DInput renamed NPN-DInput-1
- new net: D9.1 (K), OC5.1, R18.2
- new net NPN-DInput-2: OC5.4, R19.1
- new net NPN_IN-2: R18.1

Commit message: Avances en PCB
Parts:
- D3, D9: footprint PCM_Diode_SMD_AKL:D_MELF -> Diode_SMD:D_0805_2012Metric_Pad1.15x1.40mm_HandSolder
Changed lines of the file:
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@@
 			)
 		)
-		(property "Footprint" "PCM_Diode_SMD_AKL:D_MELF"
+		(property "Footprint" "Diode_SMD:D_0805_2012Metric_Pad1.15x1.40mm_HandSolder"
 			(at 83.82 115.57 0)
 			(effects
@@
 			)
 		)
-		(property "Footprint" "PCM_Diode_SMD_AKL:D_MELF"
+		(property "Footprint" "Diode_SMD:D_0805_2012Metric_Pad1.15x1.40mm_HandSolder"
 			(at 83.82 71.12 0)
 			(effects
