File: Proyecto Final/NIVARA/Imput_PNP.kicad_sch (KiCad schematic)
At the start: 0 parts

Commit message: Actualización
Parts:
- added D2: DL4007, PCM_Diode_SMD_AKL:D_MELF, symbol PCM_Diode_AKL:DL4007
- added OC2: LTV-357T-B, PCM_Package_SO_AKL:SO-4_4.4x3.9mm_P2.54mm, symbol PCM_Optocoupler_AKL:LTV-357T-B
- added R6, R7: R_0603, PCM_Resistor_SMD_AKL:R_0603_1608Metric, symbol PCM_Resistor_US_AKL:R_0603
Connections:
- new net: D2.1 (K), OC2.1, R6.2
- new net + PNP_IN +: R6.1
- new net +3.3V: OC2.4
- new net - PNP_IN -: D2.2 (A), OC2.2
- new net GND: R7.1
- new net PNP-DInput: OC2.3, R7.2

Commit message: Actualización
Parts:
- added D10: DL4007, PCM_Diode_SMD_AKL:D_MELF, symbol PCM_Diode_AKL:DL4007
- added OC6: LTV-357T-B, PCM_Package_SO_AKL:SO-4_4.4x3.9mm_P2.54mm, symbol PCM_Optocoupler_AKL:LTV-357T-B
- added R25, R26: R_0603, PCM_Resistor_SMD_AKL:R_0603_1608Metric, symbol PCM_Resistor_US_AKL:R_0603
Connections:
- net - PNP_IN - is gone; now on net GND: D2.2 (A), OC2.2
- net +3.3V: now also OC6.4
- net GND: now also D10.2 (A), OC6.2, R26.1
- net + PNP_IN + renamed PNP_IN-1
- net PNP-DInput renamed PNP-DInput-1
- new net: D10.1 (K), OC6.1, R25.2
- new net PNP-DInput-2: OC6.3, R26.2
- new net PNP_IN-2: R25.1

Commit message: Avances en PCB
Parts:
- D10, D2: footprint PCM_Diode_SMD_AKL:D_MELF -> Diode_SMD:D_0805_2012Metric_Pad1.15x1.40mm_HandSolder
Changed lines of the file:
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@@
 			)
 		)
-		(property "Footprint" "PCM_Diode_SMD_AKL:D_MELF"
+		(property "Footprint" "Diode_SMD:D_0805_2012Metric_Pad1.15x1.40mm_HandSolder"
 			(at 140.97 138.43 0)
 			(effects
@@
 			)
 		)
-		(property "Footprint" "PCM_Diode_SMD_AKL:D_MELF"
+		(property "Footprint" "Diode_SMD:D_0805_2012Metric_Pad1.15x1.40mm_HandSolder"
 			(at 140.97 88.9 0)
 			(effects
