File: Proyecto Final/NIVARA/Módulo 0-32V.kicad_sch (KiCad schematic)
At the start: 4 parts

Commit message: Avances en PCB
Parts:
- D4: footprint EasyEDA:MBF-SMD_L4.7-W3.8-P2.50-LS6.8-BL -> Puente H:MB24F-SMD_L4.7-W3.8-P2.50-LS6.8-BL
Changed lines of the file:
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@@
 			)
 		)
-		(property "Footprint" "EasyEDA:MBF-SMD_L4.7-W3.8-P2.50-LS6.8-BL"
+		(property "Footprint" "Puente H:MB24F-SMD_L4.7-W3.8-P2.50-LS6.8-BL"
 			(at 64.77 68.58 0)
 			(effects
