File: Proyecto Final/NIVARA/Módulo AOUT_010.kicad_sch (KiCad schematic)
At the start: 7 parts, among them U7 GP8201S-TC50-EW

Commit message: Avances en PCB
Parts:
- U7: footprint EasyEDA:ESOP-8_L4.9-W3.9-P1.27-LS6.0-BL-EP -> Easy Eda:GP8201S
Changed lines of the file:
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@@
 			)
 		)
-		(property "Footprint" "EasyEDA:ESOP-8_L4.9-W3.9-P1.27-LS6.0-BL-EP"
+		(property "Footprint" "Easy Eda:GP8201S"
 			(at 92.71 59.69 0)
 			(effects
