File: Proyecto Final/NIVARA/Módulo D_IN.kicad_sch (KiCad schematic)
At the start: 8 parts

Commit message: Avances en PCB
Parts:
- D6, D7: footprint PCM_Diode_SMD_AKL:D_MELF -> Diode_SMD:D_0805_2012Metric_Pad1.15x1.40mm_HandSolder
Changed lines of the file:
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@@
 			)
 		)
-		(property "Footprint" "PCM_Diode_SMD_AKL:D_MELF"
+		(property "Footprint" "Diode_SMD:D_0805_2012Metric_Pad1.15x1.40mm_HandSolder"
 			(at 69.85 110.49 0)
 			(effects
@@
 			)
 		)
-		(property "Footprint" "PCM_Diode_SMD_AKL:D_MELF"
+		(property "Footprint" "Diode_SMD:D_0805_2012Metric_Pad1.15x1.40mm_HandSolder"
 			(at 69.85 57.15 0)
 			(effects
