File: Proyecto Final/NIVARA/Módulo-DOut_NPN.kicad_sch (KiCad schematic)
At the start: 0 parts

Commit message: Actualización
Parts:
- added R27, R28: R_0603, PCM_Resistor_SMD_AKL:R_0603_1608Metric, symbol PCM_Resistor_US_AKL:R_0603
- added U6, U8: GAQY211G2S, EasyEDA:SOP-4_L4.4-W4.3-P2.54-LS6.8-BL, symbol Easy:GAQY211G2S
Connections:
- new net: R28.2, U8.1
- new net: R27.2, U6.1
- new net D_NPN_1: R27.1
- new net D_NPN_2: R28.1
- new net GND: U6.2, U6.3, U8.2, U8.3
- new net NPN_Out-1: U6.4
- new net NPN_Out-2: U8.4

Commit message: Avances en PCB
Parts:
- U6, U8: footprint EasyEDA:SOP-4_L4.4-W4.3-P2.54-LS6.8-BL -> Easy Eda:SOP-4_L4.4-W4.3-P2.54-LS6.8-BL
Changed lines of the file:
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@@
 			)
 		)
-		(property "Footprint" "EasyEDA:SOP-4_L4.4-W4.3-P2.54-LS6.8-BL"
+		(property "Footprint" "Easy Eda:SOP-4_L4.4-W4.3-P2.54-LS6.8-BL"
 			(at 167.64 128.27 0)
 			(effects
@@
 			)
 		)
-		(property "Footprint" "EasyEDA:SOP-4_L4.4-W4.3-P2.54-LS6.8-BL"
+		(property "Footprint" "Easy Eda:SOP-4_L4.4-W4.3-P2.54-LS6.8-BL"
 			(at 167.64 86.36 0)
 			(effects
