File: Proyecto Final/NIVARA/Módulo-DOut_PNP.kicad_sch (KiCad schematic)
At the start: 4 parts, among them U10 GAQY211G2S, U9 GAQY211G2S

Commit message: Avances en PCB
Parts:
- U10, U9: footprint EasyEDA:SOP-4_L4.4-W4.3-P2.54-LS6.8-BL -> Easy Eda:SOP-4_L4.4-W4.3-P2.54-LS6.8-BL
Changed lines of the file:
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@@
 			)
 		)
-		(property "Footprint" "EasyEDA:SOP-4_L4.4-W4.3-P2.54-LS6.8-BL"
+		(property "Footprint" "Easy Eda:SOP-4_L4.4-W4.3-P2.54-LS6.8-BL"
 			(at 114.3 80.01 0)
 			(effects
@@
 			)
 		)
-		(property "Footprint" "EasyEDA:SOP-4_L4.4-W4.3-P2.54-LS6.8-BL"
+		(property "Footprint" "Easy Eda:SOP-4_L4.4-W4.3-P2.54-LS6.8-BL"
 			(at 114.3 124.46 0)
 			(effects
