File: Proyecto Final/NIVARA/PowerSupply.kicad_sch (KiCad schematic)
At the start: 6 parts, among them U1 AP63203WU

Commit message: Actualización
Parts:
- added C6: C_0805, PCM_Capacitor_SMD_AKL:C_0805_2012Metric, symbol PCM_Capacitor_AKL:C_0805
- added R2, R4: R_0603, PCM_Resistor_SMD_AKL:R_0603_1608Metric, symbol PCM_Resistor_US_AKL:R_0603
Connections:
- net +3.3V: now also C6.1, R2.1; no longer U1.1 (FB)
- net GND: now also R4.2
- new net: C6.2, R2.2, R4.1, U1.1 (FB)
Other:
- moved on the sheet: C1, C5

Commit message: Actualización.
Parts:
- added JP1: SolderJumper_2_Open, symbol Jumper:SolderJumper_2_Open
- added TP1, TP2, TP3, TP4: TestPoint, symbol Connector:TestPoint
Connections:
- net +3.3V: now also JP1.2 (B), TP2.1; no longer C1.1, C5.1, C6.1, L1.2, R2.1
- net VCC: now also TP4.1
- net at C6.2, R2.2, R4.1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: now also TP1.1
- new net: C1.1, C5.1, C6.1, JP1.1 (A), L1.2, R2.1, TP3.1
Other:
- moved on the sheet: C2

Commit message: Avances en PCB
Parts:
- JP1: footprint (none) -> Jumper:SolderJumper-2_P1.3mm_Open_RoundedPad1.0x1.5mm
- TP1, TP2, TP3, TP4: footprint (none) -> TestPoint:TestPoint_Keystone_5015_Micro_Mini
Changed lines of the file:
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@@
 			)
 		)
-		(property "Footprint" ""
+		(property "Footprint" "Jumper:SolderJumper-2_P1.3mm_Open_RoundedPad1.0x1.5mm"
 			(at 129.54 39.37 0)
 			(effects
@@
 			)
 		)
-		(property "Footprint" ""
+		(property "Footprint" "TestPoint:TestPoint_Keystone_5015_Micro_Mini"
 			(at 154.94 50.8 0)
 			(effects
@@
 			)
 		)
-		(property "Footprint" ""
+		(property "Footprint" "TestPoint:TestPoint_Keystone_5015_Micro_Mini"
 			(at 59.69 44.45 0)
 			(effects
@@
 			)
 		)
-		(property "Footprint" ""
+		(property "Footprint" "TestPoint:TestPoint_Keystone_5015_Micro_Mini"
 			(at 93.98 59.69 0)
 			(effects
@@
 			)
 		)
-		(property "Footprint" ""
+		(property "Footprint" "TestPoint:TestPoint_Keystone_5015_Micro_Mini"
 			(at 132.08 36.83 0)
 			(effects
