File: Proyecto Final/NIVARA/Board_NIVARA.kicad_sch (KiCad schematic)
At the start: 3 parts, among them U2 ESP32-S3-WROOM-1

Commit message: Actualización.
Changed lines of the file:
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@@
 			)
 		)
-		(pin "RS485-A" output
+		(pin "GPIO Control" input
+			(at 242.57 48.26 180)
+			(effects
+				(font
+					(size 1.27 1.27)
+				)
+				(justify left)
+			)
+		)
+		(pin "RS485-A" bidirectional
 			(at 269.24 41.91 0)
 			(effects
@@
 			)
 		)
-		(pin "RS485-B" output
+		(pin "RS485-B" bidirectional
 			(at 269.24 44.45 0)
 			(effects
@@
 			)
 		)
-		(pin "GPIO Control" bidirectional
-			(at 269.24 48.26 0)
-			(effects
-				(font
-					(size 1.27 1.27)
-				)
-				(justify right)
-			)
-		)

Commit message: Actualización
Other:
- sheet Imput_NPN renamed Módulo_Imput_NPN
- sheet Imput_PNP renamed Módulo_Imput_PNP
- sheet RLY1 renamed Módulo - RLY
- removed sheet OutPutPNP
- removed sheet OutPut_NPN
- removed sheet RLY2
- sheet Módulo - RLY ports: added OnRLY-1, OnRLY-2, RLY1_COMÚN, RLY1_NC, RLY1_NO, RLY2_COMÚN, RLY2_NC, RLY2_NO; removed none
- sheet Módulo_Imput_NPN ports: added + NPN_IN +, - NPN_IN -, NPN-DInput; removed none
- sheet Módulo_Imput_PNP ports: added + PNP_IN +, - PNP_IN -, PNP-DInput; removed none

Commit message: Actualización
Other:
- added sheet Módulo 0-10V_IN (Módulo 0-10V_IN.kicad_sch)
- added sheet Módulo 0-32V_IN (Módulo 0-32V.kicad_sch)
- added sheet Módulo A-420-IN (Módulo A-420-IN.kicad_sch)
- added sheet Módulo AOUT_010 (Módulo AOUT_010.kicad_sch)
- added sheet Módulo D_IN (Módulo D_IN.kicad_sch)
- added sheet Módulo-AOUT_420 (Módulo-AOUT_420.kicad_sch)
- added sheet Módulo-DOut_NPN (Módulo-DOut_NPN.kicad_sch)
- sheet Módulo_Imput_NPN ports: added NPN-DInput-1, NPN-DInput-2, NPN_IN-1, NPN_IN-2; removed + NPN_IN +, - NPN_IN -, NPN-DInput
- sheet Módulo_Imput_PNP ports: added PNP-DInput-1, PNP-DInput-2, PNP_IN-1, PNP_IN-2; removed + PNP_IN +, - PNP_IN -, PNP-DInput

Commit message: Actualización
Connections:
- net DRIVER-RS485/UART_IN: now also U2.10 (GPIO17/U1TXD/ADC2_CH6); no longer U2.37 (U0TXD/GPIO43/CLK_OUT1)
- net DRIVER-RS485/UART_OUT: now also U2.11 (GPIO18/U1RXD/ADC2_CH7/CLK_OUT3); no longer U2.36 (U0RXD/GPIO44/CLK_OUT2)
- net Módulo - RLY/OnRLY-1: now also U2.18 (GPIO10/TOUCH10/ADC1_CH9/FSPICS0/FSPIIO4/SUBSPICS0)
- net Módulo - RLY/OnRLY-2: now also U2.17 (GPIO9/TOUCH9/ADC1_CH8/FSPIHD/SUBSPIHD)
- net Módulo 0-10V_IN/D_010V: now also U2.30 (SPIDQS/GPIO37/FSPIQ/SUBSPIQ)
- net Módulo 0-32V_IN/D_032V: now also U2.29 (SPIIO7/GPIO36/FSPICLK/SUBSPICLK)
- net Módulo A-420-IN/A420-OUT: now also U2.28 (SPIIO6/GPIO35/FSPID/SUBSPID)
- net Módulo AOUT_010/SCLK: now also U2.39 (GPIO1/TOUCH1/ADC1_CH0)
- net Módulo AOUT_010/SDA: now also U2.38 (GPIO2/TOUCH2/ADC1_CH1)
- net Módulo D_IN/D_InPut-1: now also U2.14 (GPIO20/U1CTS/ADC2_CH9/CLK_OUT1/USB_D+)
- net Módulo D_IN/D_InPut-2: now also U2.13 (GPIO19/U1RTS/ADC2_CH8/CLK_OUT2/USB_D-)
- net Módulo-AOUT_420/ASLK: now also U2.15 (GPIO3/TOUCH3/ADC1_CH2)
- net Módulo-AOUT_420/SDA: now also U2.4 (GPIO4/TOUCH4/ADC1_CH3)
- net Módulo_Imput_NPN/NPN-DInput-1: now also U2.19 (GPIO11/TOUCH11/ADC2_CH0/FSPID/FSPIIO5/SUBSPID)
- net Módulo_Imput_NPN/NPN-DInput-2: now also U2.20 (GPIO12/TOUCH12/ADC2_CH1/FSPICLK/FSPIIO6/SUBSPICLK)
- net Módulo_Imput_PNP/PNP-DInput-1: now also U2.21 (GPIO13/TOUCH13/ADC2_CH2/FSPIQ/FSPIIO7/SUBSPIQ)
- net Módulo_Imput_PNP/PNP-DInput-2: now also U2.22 (GPIO14/TOUCH14/ADC2_CH3/FSPIWP/FSPIDQS/SUBSPIWP)
- net Módulo-DOut_PNP/D_PNP_2: now reaches U2.12 (GPIO8/TOUCH8/ADC1_CH7/SUBSPICS1)
- net Módulo-DOut_NPN/D_NPN_1: now reaches U2.5 (GPIO5/TOUCH5/ADC1_CH4)
- net Módulo-DOut_NPN/D_NPN_2: now reaches U2.6 (GPIO6/TOUCH6/ADC1_CH5)
- net Módulo-DOut_PNP/D_PNP_1: now reaches U2.7 (GPIO7/TOUCH7/ADC1_CH6)
Other:
- added sheet Módulo-DOut_PNP (Módulo-DOut_PNP.kicad_sch)
- sheet Módulo-DOut_NPN ports: added D_NPN_1, D_NPN_2, NPN_Out-1, NPN_Out-2; removed none
- moved on the sheet: C4, R1

Commit message: Actualización de Diseño 3D e Inicio de enrutado.
Connections:
- net Módulo D_IN/D_InPut-1: now also U2.26 (GPIO45); no longer U2.14 (GPIO20/U1CTS/ADC2_CH9/CLK_OUT1/USB_D+)
- net Módulo D_IN/D_InPut-2: now also U2.16 (GPIO46); no longer U2.13 (GPIO19/U1RTS/ADC2_CH8/CLK_OUT2/USB_D-)
Changed lines of the file:
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@@
 	(wire
 		(pts
-			(xy 322.58 43.18) (xy 325.12 43.18)
+			(xy 260.35 113.03) (xy 262.89 113.03)
 		)
 		(stroke
@@
 	(wire
 		(pts
-			(xy 237.49 144.78) (xy 237.49 97.79)
+			(xy 234.95 144.78) (xy 234.95 97.79)
 		)
 		(stroke
@@
 	(wire
 		(pts
-			(xy 322.58 38.1) (xy 325.12 38.1)
+			(xy 260.35 107.95) (xy 262.89 107.95)
 		)
 		(stroke
@@
 	(wire
 		(pts
+			(xy 242.57 118.11) (xy 245.11 118.11)
+		)
+		(stroke
+			(width 0)
+			(type default)
+		)
+	)
+	(wire
+		(pts
 			(xy 298.45 86.36) (xy 298.45 72.39)
 		)
@@
 	(wire
 		(pts
+			(xy 240.03 107.95) (xy 240.03 120.65)
+		)
+		(stroke
+			(width 0)
+			(type default)
+		)
+	)
+	(wire
+		(pts
 			(xy 182.88 34.29) (xy 182.88 36.83)
 		)
@@
 	(wire
 		(pts
-			(xy 306.07 50.8) (xy 307.34 50.8)
-		)
-		(stroke
-			(width 0)
-			(type default)
-		)
-	)
-	(wire
-		(pts
 			(xy 275.59 90.17) (xy 228.6 90.17)
 		)
@@
 	(wire
 		(pts
+			(xy 240.03 120.65) (xy 245.11 120.65)
+		)
+		(stroke
+			(width 0)
+			(type default)
+		)
+	)
+	(wire
+		(pts
 			(xy 299.72 69.85) (xy 228.6 69.85)
 		)
@@
 	(wire
 		(pts
-			(xy 237.49 97.79) (xy 228.6 97.79)
+			(xy 234.95 97.79) (xy 228.6 97.79)
 		)
 		(stroke
@@
 	(wire
 		(pts
+			(xy 242.57 105.41) (xy 242.57 118.11)
+		)
+		(stroke
+			(width 0)
+			(type default)
+		)
+	)
+	(wire
+		(pts
 			(xy 293.37 99.06) (xy 285.75 99.06)
 		)
@@
 	(wire
 		(pts
-			(xy 306.07 52.07) (xy 228.6 52.07)
-		)
-		(stroke
-			(width 0)
-			(type default)
-		)
-	)
-	(wire
-		(pts
 			(xy 298.45 72.39) (xy 228.6 72.39)
 		)
@@
 	(wire
 		(pts
+			(xy 228.6 105.41) (xy 242.57 105.41)
+		)
+		(stroke
+			(width 0)
+			(type default)
+		)
+	)
+	(wire
+		(pts
 			(xy 311.15 119.38) (xy 313.69 119.38)
 		)
@@
 	(wire
 		(pts
-			(xy 306.07 50.8) (xy 306.07 52.07)
-		)
-		(stroke
-			(width 0)
-			(type default)
-		)
-	)
-	(wire
-		(pts
 			(xy 350.52 88.9) (xy 353.06 88.9)
 		)
@@
 	(wire
 		(pts
-			(xy 304.8 48.26) (xy 304.8 49.53)
-		)
-		(stroke
-			(width 0)
-			(type default)
-		)
-	)
-	(wire
-		(pts
-			(xy 304.8 49.53) (xy 228.6 49.53)
-		)
-		(stroke
-			(width 0)
-			(type default)
-		)
-	)
-	(wire
-		(pts
 			(xy 313.69 134.62) (xy 311.15 134.62)
 		)
@@
 	(wire
 		(pts
+			(xy 228.6 107.95) (xy 240.03 107.95)
+		)
+		(stroke
+			(width 0)
+			(type default)
+		)
+	)
+	(wire
+		(pts
 			(xy 313.69 105.41) (xy 311.15 105.41)
 		)
@@
 	(wire
 		(pts
-			(xy 240.03 95.25) (xy 228.6 95.25)
-		)
-		(stroke
-			(width 0)
-			(type default)
-		)
-	)
-	(wire
-		(pts
-			(xy 322.58 40.64) (xy 325.12 40.64)
+			(xy 237.49 95.25) (xy 228.6 95.25)
+		)
+		(stroke
+			(width 0)
+			(type default)
+		)
+	)
+	(wire
+		(pts
+			(xy 260.35 110.49) (xy 262.89 110.49)
 		)
 		(stroke
@@
 	(wire
 		(pts
-			(xy 240.03 142.24) (xy 240.03 95.25)
-		)
-		(stroke
-			(width 0)
-			(type default)
-		)
-	)
-	(wire
-		(pts
-			(xy 304.8 48.26) (xy 307.34 48.26)
+			(xy 237.49 142.24) (xy 237.49 95.25)
 		)
 		(stroke
@@
 	(wire
 		(pts
-			(xy 237.49 144.78) (xy 243.84 144.78)
-		)
-		(stroke
-			(width 0)
-			(type default)
-		)
-	)
-	(wire
-		(pts
-			(xy 240.03 142.24) (xy 243.84 142.24)
-		)
-		(stroke
-			(width 0)
-			(type default)
-		)
-	)
-	(wire
-		(pts
-			(xy 322.58 45.72) (xy 325.12 45.72)
+			(xy 234.95 144.78) (xy 243.84 144.78)
+		)
+		(stroke
+			(width 0)
+			(type default)
+		)
+	)
+	(wire
+		(pts
+			(xy 237.49 142.24) (xy 243.84 142.24)
+		)
+		(stroke
+			(width 0)
+			(type default)
+		)
+	)
+	(wire
+		(pts
+			(xy 260.35 115.57) (xy 262.89 115.57)
 		)
 		(stroke
@@
 	(hierarchical_label "D_IN_1+"
 		(shape input)
-		(at 325.12 38.1 0)
+		(at 262.89 107.95 0)
 		(effects
 			(font
@@
 	(hierarchical_label "D_IN_2+"
 		(shape input)
-		(at 325.12 43.18 0)
+		(at 262.89 113.03 0)
 		(effects
 			(font
@@
 	(hierarchical_label "D_IN_2-"
 		(shape input)
-		(at 325.12 45.72 0)
+		(at 262.89 115.57 0)
 		(effects
 			(font
@@
 	(hierarchical_label "D_IN_1-"
 		(shape input)
-		(at 325.12 40.64 0)
+		(at 262.89 110.49 0)
 		(effects
 			(font
@@
 	)
 	(sheet
-		(at 266.7 20.32)
+		(at 330.2 35.56)
 		(size 34.29 24.13)
 		(exclude_from_sim no)
@@
 		)
 		(property "Sheetname" "PowerSupply"
-			(at 266.192 19.304 0)
+			(at 329.692 34.544 0)
 			(effects
 				(font
@@
 		)
 		(property "Sheetfile" "PowerSupply.kicad_sch"
-			(at 266.7 37.4146 0)
+			(at 330.2 52.6546 0)
 			(effects
 				(font
@@
 	)
 	(sheet
-		(at 307.34 35.56)
+		(at 245.11 105.41)
 		(size 15.24 17.78)
 		(exclude_from_sim no)
@@
 		)
 		(property "Sheetname" "Módulo D_IN"
-			(at 307.34 34.8484 0)
+			(at 245.11 104.6984 0)
 			(effects
 				(font
@@
 		)
 		(property "Sheetfile" "Módulo D_IN.kicad_sch"
-			(at 307.34 53.9246 0)
+			(at 245.11 123.7746 0)
 			(effects
 				(font
@@
 		)
 		(pin "D_InPut-1" output
-			(at 307.34 48.26 180)
+			(at 245.11 118.11 180)
 			(effects
 				(font
@@
 		)
 		(pin "D_InPut-2" output
-			(at 307.34 50.8 180)
+			(at 245.11 120.65 180)
 			(effects
 				(font
@@
 		)
 		(pin "D_IN_1+" input
-			(at 322.58 38.1 0)
+			(at 260.35 107.95 0)
 			(effects
 				(font
@@
 		)
 		(pin "D_IN_1-" input
-			(at 322.58 40.64 0)
+			(at 260.35 110.49 0)
 			(effects
 				(font
@@
 		)
 		(pin "D_IN_2+" input
-			(at 322.58 43.18 0)
+			(at 260.35 113.03 0)
 			(effects
 				(font
@@
 		)
 		(pin "D_IN_2-" input
-			(at 322.58 45.72 0)
-			(effects
-				(font
+			(at 260.35 115.57 0)
+			(effects
+				(font
