File: Proyecto Final/NIVARA/PLC.kicad_pcb (KiCad board)
At the start: 2 copper layers, 454.9 x 92.9 mm, 18 parts, among them J1 Screw_Terminal_2_P5.00mm, J13 Screw_Terminal_4_P5.00mm, J2 Screw_Terminal_2_P5.00mm, J3 Screw_Terminal_2_P5.00mm, J4 Screw_Terminal_2_P5.00mm, J5 Screw_Terminal_6_P5.00mm, J6 Screw_Terminal_4_P5.00mm, J7 Screw_Terminal_3_P5.00mm, J8 Screw_Terminal_3_P5.00mm, J9 Screw_Terminal_2_P5.00mm, U1 AP63203WU, U2 ESP32-S3-WROOM-1

Commit message: Actualización
Parts:
- added C5: C_0805, PCM_Capacitor_SMD_AKL:C_0805_2012Metric, F.Cu at (292.5, 101.0)
- added C6: C_0805, PCM_Capacitor_SMD_AKL:C_0805_2012Metric, F.Cu at (292.5, 104.1)
- added C7: C_1206, PCM_Capacitor_SMD_AKL:C_1206_3216Metric, F.Cu at (293.2, 94.5)
- added D1: SM712, PCM_Package_TO_SOT_SMD_AKL:SOT-23, F.Cu at (298.6, 95.1)
- added R2: R_0603, PCM_Resistor_SMD_AKL:R_0603_1608Metric, F.Cu at (297.0, 100.8)
- added R4: R_0603, PCM_Resistor_SMD_AKL:R_0603_1608Metric, F.Cu at (297.0, 103.5)
- added U3: LK1802, Easy Eda:LK1802, F.Cu at (303.5, 101.6)
- added U4: ~, Package_DIP:C2992406, F.Cu at (299.6, 77.1)
Connections:
- C1 pad 1: unconnected-(C1-Pad1) -> Net-(JP1-A)
- C1 pad 2: unconnected-(C1-Pad2) -> GND
- C2 pad 1: unconnected-(C2-Pad1) -> VCC
- C2 pad 2: unconnected-(C2-Pad2) -> GND
- C3 pad 1: unconnected-(C3-Pad1) -> Net-(U1-BST)
- C3 pad 2: unconnected-(C3-Pad2) -> Net-(U1-SW)
- L1 pad 1: unconnected-(L1-Pad1) -> Net-(U1-SW)
- L1 pad 2: unconnected-(L1-Pad2) -> Net-(JP1-A)
- U1 pad 1: unconnected-(U1-FB-Pad1) -> Net-(U1-FB)
- U1 pad 2: unconnected-(U1-EN-Pad2) -> VCC
- U1 pad 3: unconnected-(U1-IN-Pad3) -> VCC
- U1 pad 4: unconnected-(U1-GND-Pad4) -> GND
- U1 pad 5: unconnected-(U1-SW-Pad5) -> Net-(U1-SW)
- U1 pad 6: unconnected-(U1-BST-Pad6) -> Net-(U1-BST)

Commit message: Avances en PCB
Parts:
- added C10: C_0805, PCM_Capacitor_SMD_AKL:C_0805_2012Metric, F.Cu at (72.5, 171.8)
- added C11: C_0603, PCM_Capacitor_SMD_AKL:C_0603_1608Metric, F.Cu at (156.0, 173.7)
- added C12: C_0603, PCM_Capacitor_SMD_AKL:C_0603_1608Metric, F.Cu at (156.0, 176.4)
- added C13: C_0603, PCM_Capacitor_SMD_AKL:C_0603_1608Metric, F.Cu at (273.7, 177.6)
- added C14: C_0603, PCM_Capacitor_SMD_AKL:C_0603_1608Metric, F.Cu at (273.7, 180.3)
- added C8: C_0805, PCM_Capacitor_SMD_AKL:C_0805_2012Metric, F.Cu at (105.8, 172.5)
- added C9: C_0603, PCM_Capacitor_SMD_AKL:C_0603_1608Metric, F.Cu at (134.0, 172.7)
- added D10: DL4007, Diode_SMD:D_0805_2012Metric_Pad1.15x1.40mm_HandSolder, F.Cu at (344.7, 141.1)
- added D2: DL4007, Diode_SMD:D_0805_2012Metric_Pad1.15x1.40mm_HandSolder, F.Cu at (344.7, 135.8)
- added D3: DL4007, Diode_SMD:D_0805_2012Metric_Pad1.15x1.40mm_HandSolder, F.Cu at (345.9, 180.7)
- added D4: MB24F_C7427849, Puente H:MB24F-SMD_L4.7-W3.8-P2.50-LS6.8-BL, F.Cu at (67.1, 169.2)
- added D5: MB24F_C7427849, Puente H:MB24F-SMD_L4.7-W3.8-P2.50-LS6.8-BL, F.Cu at (100.3, 169.9)
- added D6: DL4007, Diode_SMD:D_0805_2012Metric_Pad1.15x1.40mm_HandSolder, F.Cu at (203.7, 178.3)
- added D7: DL4007, Diode_SMD:D_0805_2012Metric_Pad1.15x1.40mm_HandSolder, F.Cu at (203.7, 183.6)
- added D8: SMF24A, PCM_Diode_SMD_AKL:D_SOD-123F, F.Cu at (163.6, 174.5)
- added D9: DL4007, Diode_SMD:D_0805_2012Metric_Pad1.15x1.40mm_HandSolder, F.Cu at (345.9, 186.0)
- added JP1: SolderJumper_2_Open, Jumper:SolderJumper-2_P1.3mm_Open_RoundedPad1.0x1.5mm, F.Cu at (274.9, 29.1)
- added K1: SRA-24VDC-CL, Easy Eda:RELAY-TH_SRA-X-CX, F.Cu at (388.4, 163.1)
- added K3: SRA-24VDC-CL, Easy Eda:RELAY-TH_SRA-X-CX, F.Cu at (388.4, 176.7)
- added OC1: LTV-357T-B, PCM_Package_SO_AKL:SO-4_4.4x3.9mm_P2.54mm, F.Cu at (336.9, 170.0)
- added OC2: LTV-357T-B, PCM_Package_SO_AKL:SO-4_4.4x3.9mm_P2.54mm, F.Cu at (335.7, 125.1)
- added OC3: LTV-357T-B, PCM_Package_SO_AKL:SO-4_4.4x3.9mm_P2.54mm, F.Cu at (194.7, 167.6)
- added OC4: LTV-357T-B, PCM_Package_SO_AKL:SO-4_4.4x3.9mm_P2.54mm, F.Cu at (194.7, 173.4)
- added OC5: LTV-357T-B, PCM_Package_SO_AKL:SO-4_4.4x3.9mm_P2.54mm, F.Cu at (336.9, 175.8)
- added OC6: LTV-357T-B, PCM_Package_SO_AKL:SO-4_4.4x3.9mm_P2.54mm, F.Cu at (335.7, 130.8)
- added R10: R_0603, PCM_Resistor_SMD_AKL:R_0603_1608Metric, F.Cu at (72.1, 168.8)
- added R11: R_0603, PCM_Resistor_SMD_AKL:R_0603_1608Metric, F.Cu at (105.4, 169.6)
- added R12: R_0603, PCM_Resistor_SMD_AKL:R_0603_1608Metric, F.Cu at (129.2, 172.7)
- added R13: R_0603, PCM_Resistor_SMD_AKL:R_0603_1608Metric, F.Cu at (201.7, 166.1)
- added R14: R_0603, PCM_Resistor_SMD_AKL:R_0603_1608Metric, F.Cu at (201.7, 168.9)
- added R15: R_0603, PCM_Resistor_SMD_AKL:R_0603_1608Metric, F.Cu at (201.7, 171.6)
- added R16: R_0603, PCM_Resistor_SMD_AKL:R_0603_1608Metric, F.Cu at (201.7, 174.3)
- added R17: R_0603, PCM_Resistor_SMD_AKL:R_0603_1608Metric, F.Cu at (162.8, 165.6)
- added R18: R_0603, PCM_Resistor_SMD_AKL:R_0603_1608Metric, F.Cu at (343.9, 174.0)
- added R19: R_0603, PCM_Resistor_SMD_AKL:R_0603_1608Metric, F.Cu at (343.9, 176.7)
- added R20: R_0603, PCM_Resistor_SMD_AKL:R_0603_1608Metric, F.Cu at (269.4, 169.5)
- added R21: R_0603, PCM_Resistor_SMD_AKL:R_0603_1608Metric, F.Cu at (269.4, 172.2)
- added R22: R_0603, PCM_Resistor_SMD_AKL:R_0603_1608Metric, F.Cu at (269.4, 174.9)
- added R23: R_0603, PCM_Resistor_SMD_AKL:R_0603_1608Metric, F.Cu at (162.8, 168.4)
- added R24: R_0603, PCM_Resistor_SMD_AKL:R_0603_1608Metric, F.Cu at (162.8, 171.1)
- added R25: R_0603, PCM_Resistor_SMD_AKL:R_0603_1608Metric, F.Cu at (342.7, 129.0)
- added R26: R_0603, PCM_Resistor_SMD_AKL:R_0603_1608Metric, F.Cu at (342.7, 131.8)
- added R27: R_0603, PCM_Resistor_SMD_AKL:R_0603_1608Metric, F.Cu at (301.1, 178.4)
- added R28: R_0603, PCM_Resistor_SMD_AKL:R_0603_1608Metric, F.Cu at (301.1, 181.1)
- added R29: R_0603, PCM_Resistor_SMD_AKL:R_0603_1608Metric, F.Cu at (232.0, 176.8)
- added R3: R_0603, PCM_Resistor_SMD_AKL:R_0603_1608Metric, F.Cu at (343.9, 168.5)
- added R30: R_0603, PCM_Resistor_SMD_AKL:R_0603_1608Metric, F.Cu at (232.0, 179.6)
- added R5: R_0603, PCM_Resistor_SMD_AKL:R_0603_1608Metric, F.Cu at (343.9, 171.3)
- added R6: R_0603, PCM_Resistor_SMD_AKL:R_0603_1608Metric, F.Cu at (342.7, 123.6)
- added R7: R_0603, PCM_Resistor_SMD_AKL:R_0603_1608Metric, F.Cu at (342.7, 126.3)
- added R8: R_0603, PCM_Resistor_SMD_AKL:R_0603_1608Metric, F.Cu at (72.1, 166.1)
- added R9: R_0603, PCM_Resistor_SMD_AKL:R_0603_1608Metric, F.Cu at (105.4, 166.8)
- added TP1: TestPoint, TestPoint:TestPoint_Keystone_5015_Micro_Mini, F.Cu at (274.5, 35.0)
- added TP2: TestPoint, TestPoint:TestPoint_Keystone_5015_Micro_Mini, F.Cu at (274.5, 38.7)
- added TP3: TestPoint, TestPoint:TestPoint_Keystone_5015_Micro_Mini, F.Cu at (274.5, 42.5)
- added TP4: TestPoint, TestPoint:TestPoint_Keystone_5015_Micro_Mini, F.Cu at (274.5, 46.2)
- added U10: GAQY211G2S, Easy Eda:SOP-4_L4.4-W4.3-P2.54-LS6.8-BL, F.Cu at (239.2, 170.5)
- added U5: GP8303-TC50-EW, Easy Eda:ESOP-10_L4.9-W3.9-P1.00-LS6.1-BL-EP, F.Cu at (274.6, 172.2)
- added U6: GAQY211G2S, Easy Eda:SOP-4_L4.4-W4.3-P2.54-LS6.8-BL, F.Cu at (302.3, 172.0)
- added U7: GP8201S-TC50-EW, Easy Eda:GP8201S, F.Cu at (157.6, 168.3)
- added U8: GAQY211G2S, Easy Eda:SOP-4_L4.4-W4.3-P2.54-LS6.8-BL, F.Cu at (308.3, 172.0)
- added U9: GAQY211G2S, Easy Eda:SOP-4_L4.4-W4.3-P2.54-LS6.8-BL, F.Cu at (233.2, 170.5)
- J2: value Screw_Terminal_2_P5.00mm -> Screw_Terminal_4_P5.00mm; footprint TerminalBlock_Phoenix:TerminalBlock_Phoenix_PT-1,5-2-5.0-H_1x02_P5.00mm_Horizontal -> TerminalBlock_Phoenix:TerminalBlock_Phoenix_PT-1,5-4-5.0-H_1x04_P5.00mm_Horizontal
- moved U4 282.1 mm to (33.0, 169.4)
- moved C7 268.3 mm to (31.7, 154.6)
- moved D1 268.3 mm to (37.1, 155.2)
- moved J13 190.6 mm to (44.0, 22.9), turned to 180 degrees
- moved J5 160.5 mm to (29.1, 97.5)
- moved J2 142.7 mm to (66.0, 22.9), turned to 180 degrees
- moved J9 138.5 mm to (113.9, 22.9), turned to 180 degrees
- moved J4 134.9 mm to (101.9, 22.9), turned to 180 degrees
- moved J3 133.2 mm to (89.9, 22.9), turned to 180 degrees
- moved J7 128.2 mm to (62.3, 97.5)
- moved J1 126.3 mm to (78.0, 22.9), turned to 180 degrees
- moved J8 112.2 mm to (80.5, 97.5)
- moved J6 98.2 mm to (98.6, 97.5)
- moved L1 97.8 mm to (260.0, 38.0)
- moved C1 96.4 mm to (267.6, 37.8)
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Connections:
- D1 pad 1: unconnected-(D1-A1-Pad1) -> GND
- D1 pad 2: unconnected-(D1-A2-Pad2) -> +3.3V
- D1 pad 3: unconnected-(D1-Com-Pad3) -> GND
- J2 pad 1: /Board_NIVARA/D_IN_2 -> /Board_NIVARA/D_IN_1+
- J2 pad 2: /Board_NIVARA/D_IN_1 -> GND
- U2 pad 10: unconnected-(U2-GPIO17/U1TXD/ADC2_CH6-Pad10) -> /Board_NIVARA/DRIVER-RS485/UART_IN
- U2 pad 11: unconnected-(U2-GPIO18/U1RXD/ADC2_CH7/CLK_OUT3-Pad11) -> /Board_NIVARA/DRIVER-RS485/UART_OUT
- U2 pad 12: unconnected-(U2-GPIO8/TOUCH8/ADC1_CH7/SUBSPICS1-Pad12) -> /Board_NIVARA/Módulo-DOut_PNP/D_PNP_2
- U2 pad 13: unconnected-(U2-GPIO19/U1RTS/ADC2_CH8/CLK_OUT2/USB_D--Pad13) -> /Board_NIVARA/Módulo D_IN/D_InPut-2
- U2 pad 14: unconnected-(U2-GPIO20/U1CTS/ADC2_CH9/CLK_OUT1/USB_D+-Pad14) -> /Board_NIVARA/Módulo D_IN/D_InPut-1
- U2 pad 15: unconnected-(U2-GPIO3/TOUCH3/ADC1_CH2-Pad15) -> /Board_NIVARA/Módulo-AOUT_420/ASLK
- U2 pad 17: unconnected-(U2-GPIO9/TOUCH9/ADC1_CH8/FSPIHD/SUBSPIHD-Pad17) -> /Board_NIVARA/Módulo - RLY/OnRLY-2
- U2 pad 18: unconnected-(U2-GPIO10/TOUCH10/ADC1_CH9/FSPICS0/FSPIIO4/SUBSPICS0-Pad18) -> /Board_NIVARA/Módulo - RLY/OnRLY-1
- U2 pad 19: unconnected-(U2-GPIO11/TOUCH11/ADC2_CH0/FSPID/FSPIIO5/SUBSPID-Pad19) -> /Board_NIVARA/Módulo_Imput_NPN/NPN-DInput-1
- U2 pad 20: unconnected-(U2-GPIO12/TOUCH12/ADC2_CH1/FSPICLK/FSPIIO6/SUBSPICLK-Pad20) -> /Board_NIVARA/Módulo_Imput_NPN/NPN-DInput-2
- U2 pad 21: unconnected-(U2-GPIO13/TOUCH13/ADC2_CH2/FSPIQ/FSPIIO7/SUBSPIQ-Pad21) -> /Board_NIVARA/Módulo_Imput_PNP/PNP-DInput-1
- U2 pad 22: unconnected-(U2-GPIO14/TOUCH14/ADC2_CH3/FSPIWP/FSPIDQS/SUBSPIWP-Pad22) -> /Board_NIVARA/Módulo_Imput_PNP/PNP-DInput-2
- U2 pad 28: unconnected-(U2-SPIIO6/GPIO35/FSPID/SUBSPID-Pad28) -> /Board_NIVARA/A420_IN1
- U2 pad 29: unconnected-(U2-SPIIO7/GPIO36/FSPICLK/SUBSPICLK-Pad29) -> /Board_NIVARA/Módulo 0-32V_IN/D_032V
- U2 pad 30: unconnected-(U2-SPIDQS/GPIO37/FSPIQ/SUBSPIQ-Pad30) -> /Board_NIVARA/Módulo 0-10V_IN/D_010V
- U2 pad 36: /Board_NIVARA/DRIVER-RS485/UART_OUT -> unconnected-(U2-U0RXD/GPIO44/CLK_OUT2-Pad36)
- U2 pad 37: /Board_NIVARA/DRIVER-RS485/UART_IN -> unconnected-(U2-U0TXD/GPIO43/CLK_OUT1-Pad37)
- U2 pad 38: unconnected-(U2-GPIO2/TOUCH2/ADC1_CH1-Pad38) -> /Board_NIVARA/Módulo AOUT_010/SDA
- U2 pad 39: unconnected-(U2-GPIO1/TOUCH1/ADC1_CH0-Pad39) -> /Board_NIVARA/Módulo AOUT_010/SCLK
- U2 pad 4: unconnected-(U2-GPIO4/TOUCH4/ADC1_CH3-Pad4) -> /Board_NIVARA/Módulo-AOUT_420/SDA
- U2 pad 5: unconnected-(U2-GPIO5/TOUCH5/ADC1_CH4-Pad5) -> /Board_NIVARA/Módulo-DOut_NPN/D_NPN_1
- U2 pad 6: unconnected-(U2-GPIO6/TOUCH6/ADC1_CH5-Pad6) -> /Board_NIVARA/Módulo-DOut_NPN/D_NPN_2
- U2 pad 7: unconnected-(U2-GPIO7/TOUCH7/ADC1_CH6-Pad7) -> /Board_NIVARA/Módulo-DOut_PNP/D_PNP_1
- U3 pad 1: unconnected-(U3-1C-Pad1) -> Net-(U3-1C)
- U3 pad 2: unconnected-(U3-E-Pad2) -> GND
- U3 pad 3: unconnected-(U3-1B-Pad3) -> /Board_NIVARA/Módulo - RLY/OnRLY-1
- U3 pad 4: unconnected-(U3-2B-Pad4) -> /Board_NIVARA/Módulo - RLY/OnRLY-2
- U3 pad 5: unconnected-(U3-COM-Pad5) -> VCC
- U3 pad 6: unconnected-(U3-2C-Pad6) -> Net-(U3-2C)
Other:
- board size 454.9 x 92.9 mm -> 558.8 x 96.7 mm

Commit message: Actualización de Diseño 3D e Inicio de enrutado.
Parts:
- added REF**: MountingHole_2.5mm, MountingHole:MountingHole_2.5mm, F.Cu at (28.8, 85.1)
- added REF**: MountingHole_2.5mm, MountingHole:MountingHole_2.5mm, F.Cu at (113.9, 35.1)
- moved K3 371.2 mm to (32.3, 71.8), turned to -90 degrees
- moved K1 350.9 mm to (47.2, 80.8), turned to -90 degrees
- moved U3 350.7 mm to (45.3, 65.3)
- moved D3 320.6 mm to (55.4, 45.2)
- moved R3 310.8 mm to (64.8, 32.0)
- moved OC1 310.7 mm to (57.9, 33.5)
- moved R5 310.5 mm to (64.8, 35.2)
- moved R18 310.3 mm to (64.8, 38.4)
- moved OC5 310.2 mm to (58.0, 40.1)
- moved R19 310.0 mm to (64.9, 41.7)
- moved D9 297.3 mm to (78.5, 56.2)
- moved R6 293.4 mm to (59.9, 45.2)
- moved D10 290.7 mm to (70.4, 44.9)
- moved D2 283.5 mm to (76.2, 44.9)
- moved R7 278.9 mm to (79.8, 33.3)
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Connections:
- U2 pad 13: /Board_NIVARA/Módulo D_IN/D_InPut-2 -> unconnected-(U2-GPIO19/U1RTS/ADC2_CH8/CLK_OUT2/USB_D--Pad13)
- U2 pad 14: /Board_NIVARA/Módulo D_IN/D_InPut-1 -> unconnected-(U2-GPIO20/U1CTS/ADC2_CH9/CLK_OUT1/USB_D+-Pad14)
- U2 pad 16: unconnected-(U2-GPIO46-Pad16) -> /Board_NIVARA/Módulo D_IN/D_InPut-2
- U2 pad 26: unconnected-(U2-GPIO45-Pad26) -> /Board_NIVARA/Módulo D_IN/D_InPut-1
Routing:
- net GND: track 0.00 -> 657.5 mm, vias 0 -> 5
- net +3.3V: track 0.00 -> 253.2 mm, vias 0 -> 8
- net VCC: track 0.00 -> 174.1 mm, vias 0 -> 3
- net /Board_NIVARA/A420_IN1: track 0.00 -> 135.9 mm, vias 0 -> 1
- net /Board_NIVARA/Módulo 0-32V_IN/D_032V: track 0.00 -> 135.1 mm, vias 0 -> 2
- net /Board_NIVARA/Módulo 0-10V_IN/D_010V: track 0.00 -> 117.7 mm, vias 0 -> 2
- net /Board_NIVARA/Módulo AOUT_010/SCLK: track 0.00 -> 96.7 mm, vias 0 -> 3
- net /Board_NIVARA/Módulo_Imput_NPN/NPN-DInput-2: track 0.00 -> 75.8 mm, vias 0 -> 2
- net /Board_NIVARA/Módulo_Imput_NPN/NPN-DInput-1: track 0.00 -> 75.6 mm, vias 0 -> 2
- net /Board_NIVARA/D_IN_2+: track 0.00 -> 69.3 mm
- net /Board_NIVARA/Módulo D_IN/D_InPut-1: track 0.00 -> 67.9 mm, vias 0 -> 2
- net /Board_NIVARA/Módulo_Imput_PNP/PNP-DInput-1: track 0.00 -> 65.3 mm, vias 0 -> 2
- net /Board_NIVARA/Módulo_Imput_PNP/PNP-DInput-2: track 0.00 -> 62.6 mm, vias 0 -> 2
- net /Board_NIVARA/Módulo - RLY/OnRLY-2: track 0.00 -> 61.4 mm
- net /Board_NIVARA/Módulo AOUT_010/SDA: track 0.00 -> 60.1 mm, vias 0 -> 4
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Other:
- board size 558.8 x 96.7 mm -> 101.2 x 82 mm
